Commit message: tasks configured

File: sim/object_descriptions/urdf/objects/table.urdf.xacro (robot description, xacro)
@@ -8,23 +8,56 @@
   <xacro:arg name="w" default="0.5" />
   <xacro:arg name="color" default="blue" />
+  <xacro:property name="h" value="$(arg h)" />
+  <xacro:property name="l" value="$(arg l)" />
+  <xacro:property name="w" value="$(arg w)" />
   <link name="table">
+    <collision>
+      <origin xyz="0 0 ${h/2}" rpy="0 0 0"/>
+      <geometry>
+        <box size="${l} ${w} ${h}"/>
+      </geometry>
+    </collision>
+    <visual>
+      <origin xyz="0 0 ${h/2}" rpy="0 0 0"/>
+      <geometry>
+        <box size="${l} ${w} ${h}"/>
+      </geometry>
+    </visual>
+    <surface>
+    <friction>
+      <ode>
+        <mu>100</mu>
+        <mu2>100</mu2>
+      </ode>
+    </friction>
+  </surface>
     <inertial>
-      <origin xyz="$(arg x) $(arg y) $(arg z)" />
-      <mass value="10.0" />
-      <inertia ixx="10.0" ixy="0.0" ixz="0.0" iyy="10.0" iyz="0.0" izz="10.0" />
+      <origin xyz="0 0 ${h/2}" rpy="0 0 0"/>
+      <mass value="10"/>
+      <inertia
+        ixx="10.0" ixy="0.0" ixz="0.0"
+        iyy="10.0" iyz="0.0"
+        izz="10.0"/>
     </inertial>
-    <visual>
-      <origin xyz="$(arg x) $(arg y) $(arg z)" />
-      <geometry>
+  </link>
+  <!-- <link name="table">
+    <inertial> -->
+      <!-- <origin xyz="$(arg x) $(arg y) $(arg z)" /> -->
+      <!-- <mass value="10.0" /> -->
+      <!-- <inertia ixx="1.0" ixy="0.0" ixz="0.0" iyy="1.0" iyz="0.0" izz="1.0" /> -->
+    <!-- </inertial>
+    <visual> -->
+      <!-- <origin xyz="$(arg x) $(arg y) $(arg z)" /> -->
+      <!-- <geometry>
         <box size="$(arg l) $(arg w) $(arg h)" />
       </geometry>
     </visual>
-    <collision>
-      <origin xyz="$(arg x) $(arg y) $(arg z)" />
-      <geometry>
+    <collision> -->
+      <!-- <origin xyz="$(arg x) $(arg y) $(arg z)" /> -->
+      <!-- <geometry>
         <box size="$(arg l) $(arg w) $(arg h)" />
       </geometry>
-    </collision>
-    <surface>
+    </collision> -->
+    <!-- <surface>
       <friction>
         <ode>
@@ -33,7 +66,8 @@
         </ode>
       </friction>
-    </surface>
-  </link>
+    </surface> -->
+  <!-- </link> -->
   <gazebo reference="table">
+     <!-- <origin xyz="$(arg x) $(arg y) $(arg z)" /> -->
     <visual>
       <material>
@@ -41,5 +75,15 @@
         <xacro:color color="$(arg color)" />
       </material>
+      <!-- <origin xyz="$(arg x) $(arg y) $(arg z)" /> -->
+      <!-- <geometry>
+        <box size="$(arg l) $(arg w) $(arg h)" />
+      </geometry> -->
     </visual>
+    <dampingFactor>0.005</dampingFactor>
+    <kp>1000000</kp>
+    <kd>1.0</kd>
+    <mu1>1000.0</mu1>
+    <mu2>1000.0</mu2>
+    <minDepth>0.001</minDepth>
   </gazebo>
 </robot>

Commit message: fixes to sim and world environments

File: sim/object_descriptions/urdf/objects/table.urdf.xacro (robot description, xacro)
@@ -9,17 +9,15 @@
   <xacro:arg name="color" default="blue" />
   <xacro:property name="h" value="$(arg h)" />
-  <xacro:property name="l" value="$(arg l)" />
-  <xacro:property name="w" value="$(arg w)" />
   <link name="table">
     <collision>
-      <origin xyz="0 0 ${h/2}" rpy="0 0 0"/>
+      <origin xyz="0 0 ${h/2.0}" rpy="0 0 0"/>
       <geometry>
-        <box size="${l} ${w} ${h}"/>
+        <box size="$(arg l) $(arg w) $(arg h)"/>
       </geometry>
     </collision>
     <visual>
-      <origin xyz="0 0 ${h/2}" rpy="0 0 0"/>
+      <origin xyz="0 0 ${h/2.0}" rpy="0 0 0"/>
       <geometry>
-        <box size="${l} ${w} ${h}"/>
+        <box size="$(arg l) $(arg w) $(arg h)"/>
       </geometry>
     </visual>
@@ -32,12 +30,12 @@
     </friction>
   </surface>
-    <inertial>
-      <origin xyz="0 0 ${h/2}" rpy="0 0 0"/>
-      <mass value="10"/>
-      <inertia
-        ixx="10.0" ixy="0.0" ixz="0.0"
-        iyy="10.0" iyz="0.0"
-        izz="10.0"/>
-    </inertial>
+  <inertial>
+    <origin xyz="0 0 0" rpy="0 0 0"/>
+    <mass value="10"/>
+    <inertia
+      ixx="0.24" ixy="0.0" ixz="0.0"
+      iyy="0.166" iyz="0.0"
+      izz="0.34"/>
+  </inertial>
   </link>
   <!-- <link name="table">
