Commit message: refactor

File: ros2_agents/robots/locobot_wx250s/control/sim/gz_control.urdf.xacro (robot description, xacro)
@@ -101,5 +101,5 @@
       <robot_param>robot_description</robot_param>
       <parameters>
-        $(find ros2_transformers)/robots/locobot_wx250s/control/ros_controllers.yaml
+        $(find ros2_agents)/robots/locobot_wx250s/control/ros_controllers.yaml
       </parameters>
     </plugin>

File: ros2_agents/robots/locobot_wx250s/description/urdf/arms/mobile_arm.urdf.xacro (robot description, xacro)
@@ -7,5 +7,5 @@
         <child link="${robot_name}_arm_base_link"/>
       </joint>
-    <xacro:include filename="$(find ros2_transformers)/robots/locobot_wx250s/description/urdf/arms/mobile_wx250s.urdf.xacro"/>
+    <xacro:include filename="$(find ros2_agents)/robots/locobot_wx250s/description/urdf/arms/mobile_wx250s.urdf.xacro"/>
     <gazebo reference="${robot_name}_arm_base_link">
       <material>Gazebo/DarkGrey</material>

File: ros2_agents/robots/locobot_wx250s/description/urdf/arms/mobile_wx250s.urdf.xacro (robot description, xacro)
@@ -5,9 +5,9 @@
     scope="global" />
   <xacro:property name="mesh_directory"
-    value="package://ros2_transformers/robots/locobot_wx250s/description/meshes/arms" />
+    value="package://ros2_agents/robots/locobot_wx250s/description/meshes/arms" />
   <xacro:property name="pi_offset" value="0.00001" />
   <xacro:property name="initial_positions_file" default="$(find interbotix_xslocobot_sim)/config/initial_positions.yaml" />
   <xacro:property name="initial_positions" default="${xacro.load_yaml(initial_positions_file)}" />
-  <xacro:include filename="$(find ros2_transformers)/robots/locobot_wx250s/description/urdf/arms/ar_tag.urdf.xacro" />
+  <xacro:include filename="$(find ros2_agents)/robots/locobot_wx250s/description/urdf/arms/ar_tag.urdf.xacro" />
   <link name="${robot_name}_arm_base_link">
     <visual>
@@ -695,5 +695,5 @@
             <material>
               <xacro:include
-                filename="$(find ros2_transformers)/robots/locobot_wx250s/description/urdf/colors.urdf.xacro" />
+                filename="$(find ros2_agents)/robots/locobot_wx250s/description/urdf/colors.urdf.xacro" />
               <xacro:color color="black" />
             </material>
@@ -704,5 +704,5 @@
             <material>
               <xacro:include
-                filename="$(find ros2_transformers)/robots/locobot_wx250s/description/urdf/colors.urdf.xacro" />
+                filename="$(find ros2_agents)/robots/locobot_wx250s/description/urdf/colors.urdf.xacro" />
               <xacro:color color="black" />
             </material>
@@ -713,5 +713,5 @@
             <material>
               <xacro:include
-                filename="$(find ros2_transformers)/robots/locobot_wx250s/description/urdf/colors.urdf.xacro" />
+                filename="$(find ros2_agents)/robots/locobot_wx250s/description/urdf/colors.urdf.xacro" />
               <xacro:color color="black" />
             </material>
@@ -722,5 +722,5 @@
             <material>
               <xacro:include
-                filename="$(find ros2_transformers)/robots/locobot_wx250s/description/urdf/colors.urdf.xacro" />
+                filename="$(find ros2_agents)/robots/locobot_wx250s/description/urdf/colors.urdf.xacro" />
               <xacro:color color="black" />
             </material>
@@ -731,5 +731,5 @@
             <material>
               <xacro:include
-                filename="$(find ros2_transformers)/robots/locobot_wx250s/description/urdf/colors.urdf.xacro" />
+                filename="$(find ros2_agents)/robots/locobot_wx250s/description/urdf/colors.urdf.xacro" />
               <xacro:color color="black" />
             </material>
@@ -740,5 +740,5 @@
             <material>
               <xacro:include
-                filename="$(find ros2_transformers)/robots/locobot_wx250s/description/urdf/colors.urdf.xacro" />
+                filename="$(find ros2_agents)/robots/locobot_wx250s/description/urdf/colors.urdf.xacro" />
               <xacro:color color="black" />
             </material>
@@ -749,5 +749,5 @@
             <material>
               <xacro:include
-                filename="$(find ros2_transformers)/robots/locobot_wx250s/description/urdf/colors.urdf.xacro" />
+                filename="$(find ros2_agents)/robots/locobot_wx250s/description/urdf/colors.urdf.xacro" />
               <xacro:color color="black" />
             </material>
@@ -758,5 +758,5 @@
             <material>
               <xacro:include
-                filename="$(find ros2_transformers)/robots/locobot_wx250s/description/urdf/colors.urdf.xacro" />
+                filename="$(find ros2_agents)/robots/locobot_wx250s/description/urdf/colors.urdf.xacro" />
               <xacro:color color="black" />
             </material>
@@ -767,5 +767,5 @@
             <material>
               <xacro:include
-                filename="$(find ros2_transformers)/robots/locobot_wx250s/description/urdf/colors.urdf.xacro" />
+                filename="$(find ros2_agents)/robots/locobot_wx250s/description/urdf/colors.urdf.xacro" />
               <xacro:color color="black" />
             </material>
@@ -776,5 +776,5 @@
             <material>
               <xacro:include
-                filename="$(find ros2_transformers)/robots/locobot_wx250s/description/urdf/colors.urdf.xacro" />
+                filename="$(find ros2_agents)/robots/locobot_wx250s/description/urdf/colors.urdf.xacro" />
               <xacro:color color="black" />
             </material>
@@ -785,5 +785,5 @@
             <material>
               <xacro:include
-                filename="$(find ros2_transformers)/robots/locobot_wx250s/description/urdf/colors.urdf.xacro" />
+                filename="$(find ros2_agents)/robots/locobot_wx250s/description/urdf/colors.urdf.xacro" />
               <xacro:color color="black" />
             </material>
@@ -794,5 +794,5 @@
             <material>
               <xacro:include
-                filename="$(find ros2_transformers)/robots/locobot_wx250s/description/urdf/colors.urdf.xacro" />
+                filename="$(find ros2_agents)/robots/locobot_wx250s/description/urdf/colors.urdf.xacro" />
               <xacro:color color="black" />
             </material>
@@ -803,5 +803,5 @@
             <material>
               <xacro:include
-                filename="$(find ros2_transformers)/robots/locobot_wx250s/description/urdf/colors.urdf.xacro" />
+                filename="$(find ros2_agents)/robots/locobot_wx250s/description/urdf/colors.urdf.xacro" />
               <xacro:color color="black" />
             </material>
@@ -812,5 +812,5 @@
             <material>
               <xacro:include
-                filename="$(find ros2_transformers)/robots/locobot_wx250s/description/urdf/colors.urdf.xacro" />
+                filename="$(find ros2_agents)/robots/locobot_wx250s/description/urdf/colors.urdf.xacro" />
               <xacro:color color="black" />
             </material>
@@ -821,5 +821,5 @@
             <material>
               <xacro:include
-                filename="$(find ros2_transformers)/robots/locobot_wx250s/description/urdf/colors.urdf.xacro" />
+                filename="$(find ros2_agents)/robots/locobot_wx250s/description/urdf/colors.urdf.xacro" />
               <xacro:color color="black" />
             </material>
@@ -830,5 +830,5 @@
             <material>
               <xacro:include
-                filename="$(find ros2_transformers)/robots/locobot_wx250s/description/urdf/colors.urdf.xacro" />
+                filename="$(find ros2_agents)/robots/locobot_wx250s/description/urdf/colors.urdf.xacro" />
               <xacro:color color="black" />
             </material>

File: ros2_agents/robots/locobot_wx250s/description/urdf/base/kobuki.urdf.xacro (robot description, xacro)
@@ -61,5 +61,5 @@
       <geometry>
         <mesh
-          filename="package://ros2_transformers/robots/locobot_wx250s/description/meshes/base/kobuki.dae"/>
+          filename="package://ros2_agents/robots/locobot_wx250s/description/meshes/base/kobuki.dae"/>
       </geometry>
     </visual>
@@ -129,5 +129,5 @@
       <geometry>
         <mesh
-          filename="package://ros2_transformers/robots/locobot_wx250s/description/meshes/base/kobuki_wheel.dae"/>
+          filename="package://ros2_agents/robots/locobot_wx250s/description/meshes/base/kobuki_wheel.dae"/>
       </geometry>
     </visual>
@@ -192,5 +192,5 @@
       <geometry>
         <mesh
-          filename="package://ros2_transformers/robots/locobot_wx250s/description/meshes/base/kobuki_wheel.dae"/>
+          filename="package://ros2_agents/robots/locobot_wx250s/description/meshes/base/kobuki_wheel.dae"/>
       </geometry>
     </visual>

File: ros2_agents/robots/locobot_wx250s/description/urdf/body/camera_tower.urdf.xacro (robot description, xacro)
@@ -16,5 +16,5 @@
         <geometry>
           <mesh
-            filename="package://ros2_transformers/robots/locobot_wx250s/description/meshes/body/locobot_camera_tower_large.stl"
+            filename="package://ros2_agents/robots/locobot_wx250s/description/meshes/body/locobot_camera_tower_large.stl"
             scale="${mesh_scale}"/>
         </geometry>
@@ -27,5 +27,5 @@
         <geometry>
           <mesh
-            filename="package://ros2_transformers/robots/locobot_wx250s/description/meshes/body/locobot_camera_tower_large_simple.stl"
+            filename="package://ros2_agents/robots/locobot_wx250s/description/meshes/body/locobot_camera_tower_large_simple.stl"
             scale="${mesh_scale}"/>
         </geometry>

File: ros2_agents/robots/locobot_wx250s/description/urdf/body/pan_and_tilt.urdf.xacro (robot description, xacro)
@@ -27,5 +27,5 @@
         <geometry>
           <mesh
-            filename="package://ros2_transformers/robots/locobot_wx250s/description/meshes/body/locobot_pan.stl"
+            filename="package://ros2_agents/robots/locobot_wx250s/description/meshes/body/locobot_pan.stl"
             scale="0.001 0.001 0.001" />
         </geometry>
@@ -38,5 +38,5 @@
         <geometry>
           <mesh
-            filename="package://ros2_transformers/robots/locobot_wx250s/description/meshes/body/locobot_pan.stl"
+            filename="package://ros2_agents/robots/locobot_wx250s/description/meshes/body/locobot_pan.stl"
             scale="0.001 0.001 0.001" />
         </geometry>
@@ -85,5 +85,5 @@
         <geometry>
           <mesh
-            filename="package://ros2_transformers/robots/locobot_wx250s/description/meshes/body/locobot_tilt.stl"
+            filename="package://ros2_agents/robots/locobot_wx250s/description/meshes/body/locobot_tilt.stl"
             scale="0.001 0.001 0.001" />
         </geometry>
@@ -96,5 +96,5 @@
         <geometry>
           <mesh
-            filename="package://ros2_transformers/robots/locobot_wx250s/description/meshes/body/locobot_tilt.stl"
+            filename="package://ros2_agents/robots/locobot_wx250s/description/meshes/body/locobot_tilt.stl"
             scale="0.001 0.001 0.001" />
         </geometry>
@@ -137,5 +137,5 @@
         <geometry>
           <mesh
-            filename="package://ros2_transformers/robots/locobot_wx250s/description/meshes/locobot_camera.stl"
+            filename="package://ros2_agents/robots/locobot_wx250s/description/meshes/locobot_camera.stl"
             scale="0.001 0.001 0.001" />
         </geometry>
@@ -151,5 +151,5 @@
         <geometry>
           <mesh
-            filename="package://ros2_transformers/robots/locobot_wx250s/description/meshes/locobot_camera.stl"
+            filename="package://ros2_agents/robots/locobot_wx250s/description/meshes/locobot_camera.stl"
             scale="0.001 0.001 0.001" />
         </geometry>

File: ros2_agents/robots/locobot_wx250s/description/urdf/body/plate.urdf.xacro (robot description, xacro)
@@ -16,5 +16,5 @@
         <geometry>
           <mesh
-            filename="package://ros2_transformers/robots/locobot_wx250s/description/meshes/base/locobot_base_plate.stl"
+            filename="package://ros2_agents/robots/locobot_wx250s/description/meshes/base/locobot_base_plate.stl"
             scale="${mesh_scale}"/>
         </geometry>
@@ -27,5 +27,5 @@
         <geometry>
           <mesh
-            filename="package://ros2_transformers/robots/locobot_wx250s/description/meshes/base/locobot_base_plate.stl"
+            filename="package://ros2_agents/robots/locobot_wx250s/description/meshes/base/locobot_base_plate.stl"
             scale="${mesh_scale}"/>
         </geometry>

File: ros2_agents/robots/locobot_wx250s/description/urdf/locobot.urdf.xacro (robot description, xacro)
@@ -36,21 +36,21 @@
   <xacro:property name="finger_limit_vel" value="1.0" />
   <xacro:arg name="initial_positions_file"
-    default="$(find ros2_transformers)/robots/locobot_wx250s/control/sim/initial_positions.yaml" />
+    default="$(find ros2_agents)/robots/locobot_wx250s/control/sim/initial_positions.yaml" />
   <xacro:property name="initial_positions_file" default="$(arg initial_positions_file)" />
   <xacro:property name="initial_positions" default="${xacro.load_yaml(initial_positions_file)}" />
   <material name="interbotix_black">
     <texture
-      filename="package://ros2_transformers/robots/locobot_wx250s/description/images/interbotix_black.png" />
+      filename="package://ros2_agents/robots/locobot_wx250s/description/images/interbotix_black.png" />
   </material>
-  <xacro:include filename="$(find ros2_transformers)/robots/locobot_wx250s/description/urdf/body/plate.urdf.xacro" />
-  <xacro:include filename="$(find ros2_transformers)/robots/locobot_wx250s/description/urdf/body/battery.urdf.xacro" />
-  <xacro:include filename="$(find ros2_transformers)/robots/locobot_wx250s/description/urdf/body/camera_tower.urdf.xacro" />
-  <xacro:include filename="$(find ros2_transformers)/robots/locobot_wx250s/description/urdf/body/pan_and_tilt.urdf.xacro" />
+  <xacro:include filename="$(find ros2_agents)/robots/locobot_wx250s/description/urdf/body/plate.urdf.xacro" />
+  <xacro:include filename="$(find ros2_agents)/robots/locobot_wx250s/description/urdf/body/battery.urdf.xacro" />
+  <xacro:include filename="$(find ros2_agents)/robots/locobot_wx250s/description/urdf/body/camera_tower.urdf.xacro" />
+  <xacro:include filename="$(find ros2_agents)/robots/locobot_wx250s/description/urdf/body/pan_and_tilt.urdf.xacro" />
     <xacro:include
-      filename="$(find ros2_transformers)/robots/locobot_wx250s/description/urdf/base/kobuki.urdf.xacro" />
+      filename="$(find ros2_agents)/robots/locobot_wx250s/description/urdf/base/kobuki.urdf.xacro" />
     <xacro:property name="mesh_scale" value="0.001 0.001 0.001" />
   <!-- ********************************** Arm ********************************** -->
   <xacro:include
-  filename="$(find ros2_transformers)/robots/locobot_wx250s/description/urdf/arms/mobile_arm.urdf.xacro" />
+  filename="$(find ros2_agents)/robots/locobot_wx250s/description/urdf/arms/mobile_arm.urdf.xacro" />
 <xacro:mobile_arm />
   <!-- ********************************** Body **********************************  -->
@@ -101,6 +101,6 @@
           xyz="0.047228 0 0.44425" />
       </xacro:pan_and_tilt>
-  <xacro:include filename="$(find ros2_transformers)/robots/locobot_wx250s/control/sim/gz_control.urdf.xacro" />
-  <xacro:include filename="$(find ros2_transformers)/robots/locobot_wx250s/control/sim/gz_sense.urdf.xacro" />
+  <xacro:include filename="$(find ros2_agents)/robots/locobot_wx250s/control/sim/gz_control.urdf.xacro" />
+  <xacro:include filename="$(find ros2_agents)/robots/locobot_wx250s/control/sim/gz_sense.urdf.xacro" />
   <gazebo>
     <xacro:fake_actuators />

File: ros2_agents/sim/object_descriptions/urdf/camera/camera.urdf.xacro (robot description, xacro)
@@ -2,5 +2,5 @@
 <robot name="camera" xmlns:xacro="http://ros.org/wiki/xacro">
   <link name="world"/>
-  <xacro:include filename="$(find ros2_transformers)/urdf/camera/camera_macro.urdf.xacro"/>
+  <xacro:include filename="$(find ros2_agents)/urdf/camera/camera_macro.urdf.xacro"/>
   <!-- camera side view for the cylinder -->
   <!-- <xacro:kinect_camera parent_link="world" cam_py="-0.25" cam_pz="0.04"/> -->

File: ros2_agents/sim/object_descriptions/urdf/camera/camera_macro.urdf.xacro (robot description, xacro)
@@ -7,5 +7,5 @@
         <origin xyz="0 0 0" rpy="0 0 ${M_PI/2}"/>
         <geometry>
-          <mesh filename="package://ros2_transformers/meshes/camera/kinect.dae"/>
+          <mesh filename="package://ros2_agents/meshes/camera/kinect.dae"/>
         </geometry>
       </visual>
@@ -13,5 +13,5 @@
         <origin xyz="0 0 0" rpy="0 0 ${M_PI/2}"/>
         <geometry>
-          <mesh filename="package://ros2_transformers/meshes/camera/kinect.dae"/>
+          <mesh filename="package://ros2_agents/meshes/camera/kinect.dae"/>
         </geometry>
       </collision>

File: ros2_agents/sim/object_descriptions/urdf/objects/barclamp.urdf.xacro (robot description, xacro)
@@ -9,5 +9,5 @@
       <origin xyz="$(arg x) $(arg y) $(arg z)" />
       <geometry>
-        <mesh filename="$(find ros2_transformers)/meshes/objects/bar_clamp.dae" />
+        <mesh filename="$(find ros2_agents)/meshes/objects/bar_clamp.dae" />
 	    </geometry>
     </visual>
@@ -15,5 +15,5 @@
       <origin xyz="$(arg x) $(arg y) $(arg z)" />
       <geometry>
-        <mesh filename="$(find ros2_transformers)/meshes/objects/bar_clamp.dae" />
+        <mesh filename="$(find ros2_agents)/meshes/objects/bar_clamp.dae" />
 	    </geometry>
     </collision>
@@ -26,5 +26,5 @@
     <visual>
       <material>
-        <xacro:include filename="$(find ros2_transformers)/tasks/sim/object_descriptions/urdf/colors.urdf.xacro" />
+        <xacro:include filename="$(find ros2_agents)/tasks/sim/object_descriptions/urdf/colors.urdf.xacro" />
         <xacro:color color="$(arg color)" />
       </material>

File: ros2_agents/sim/object_descriptions/urdf/objects/block.urdf.xacro (robot description, xacro)
@@ -33,5 +33,5 @@
         <visual>
             <material>
-                <xacro:include filename="$(find ros2_transformers)/sim/object_descriptions/urdf/colors.urdf.xacro" />
+                <xacro:include filename="$(find ros2_agents)/sim/object_descriptions/urdf/colors.urdf.xacro" />
                 <xacro:color color="$(arg color)" />
             </material>

File: ros2_agents/sim/object_descriptions/urdf/objects/bowl.urdf.xacro (robot description, xacro)
@@ -4,10 +4,10 @@
   <visual>
     <geometry>
-	    <mesh filename="package://ros2_transformers/meshes/objects/bowl.dae"/>
+	    <mesh filename="package://ros2_agents/meshes/objects/bowl.dae"/>
 	</geometry>
   </visual>
   <collision>
     <geometry>
-       <mesh filename="package://ros2_transformers/meshes/objects/bowl.dae"/>
+       <mesh filename="package://ros2_agents/meshes/objects/bowl.dae"/>
 	</geometry>
   </collision>

File: ros2_agents/sim/object_descriptions/urdf/objects/strawberry.urdf.xacro (robot description, xacro)
@@ -4,10 +4,10 @@
   <visual>
      <geometry>
-	       <mesh filename="package://ros2_transformers/meshes/objects/strawberry.dae"/>
+	       <mesh filename="package://ros2_agents/meshes/objects/strawberry.dae"/>
 	     </geometry>
   </visual>
   <collision>
     <geometry>
-       <mesh filename="package://ros2_transformers/meshes/objects/strawberry.dae"/>
+       <mesh filename="package://ros2_agents/meshes/objects/strawberry.dae"/>
 	   </geometry>
   </collision>

File: ros2_agents/sim/object_descriptions/urdf/objects/table.urdf.xacro (robot description, xacro)
@@ -70,5 +70,5 @@
     <visual>
       <material>
-        <xacro:include filename="$(find ros2_transformers)/sim/object_descriptions/urdf/colors.urdf.xacro" />
+        <xacro:include filename="$(find ros2_agents)/sim/object_descriptions/urdf/colors.urdf.xacro" />
         <xacro:color color="$(arg color)" />
       </material>

File: ros2_agents/sim/object_descriptions/urdf/robots/panda_camera.urdf.xacro (robot description, xacro)
@@ -3,5 +3,5 @@
   <!-- Panda Arm + Hand -->
   <!-- <xacro:include filename="$(find franka_description)/robots/panda_arm_hand.urdf.xacro"/> -->
-  <xacro:include filename="$(find ros2_transformers)/urdf/camera/camera_macro.urdf.xacro"/>
+  <xacro:include filename="$(find ros2_agents)/urdf/camera/camera_macro.urdf.xacro"/>
   <!-- camera side view for the cylinder -->
   <xacro:kinect_camera parent_link="locobot_base_footprint" cam_py="-0.25" cam_pz="0.04"/>
