Commit message: fix z command bug and added licenses

File: ros2_agents/sim/object_descriptions/urdf/objects/table.urdf.xacro (robot description, xacro)
@@ -22,12 +22,4 @@
       </geometry>
     </visual>
-    <surface>
-    <friction>
-      <ode>
-        <mu>100</mu>
-        <mu2>100</mu2>
-      </ode>
-    </friction>
-  </surface>
   <inertial>
     <origin xyz="0 0 0" rpy="0 0 0"/>
@@ -39,33 +31,5 @@
   </inertial>
   </link>
-  <!-- <link name="table">
-    <inertial> -->
-      <!-- <origin xyz="$(arg x) $(arg y) $(arg z)" /> -->
-      <!-- <mass value="10.0" /> -->
-      <!-- <inertia ixx="1.0" ixy="0.0" ixz="0.0" iyy="1.0" iyz="0.0" izz="1.0" /> -->
-    <!-- </inertial>
-    <visual> -->
-      <!-- <origin xyz="$(arg x) $(arg y) $(arg z)" /> -->
-      <!-- <geometry>
-        <box size="$(arg l) $(arg w) $(arg h)" />
-      </geometry>
-    </visual>
-    <collision> -->
-      <!-- <origin xyz="$(arg x) $(arg y) $(arg z)" /> -->
-      <!-- <geometry>
-        <box size="$(arg l) $(arg w) $(arg h)" />
-      </geometry>
-    </collision> -->
-    <!-- <surface>
-      <friction>
-        <ode>
-          <mu>100</mu>
-          <mu2>100</mu2>
-        </ode>
-      </friction>
-    </surface> -->
-  <!-- </link> -->
   <gazebo reference="table">
-     <!-- <origin xyz="$(arg x) $(arg y) $(arg z)" /> -->
     <visual>
       <material>
@@ -73,15 +37,5 @@
         <xacro:color color="$(arg color)" />
       </material>
-      <!-- <origin xyz="$(arg x) $(arg y) $(arg z)" /> -->
-      <!-- <geometry>
-        <box size="$(arg l) $(arg w) $(arg h)" />
-      </geometry> -->
     </visual>
-    <dampingFactor>0.005</dampingFactor>
-    <kp>1000000</kp>
-    <kd>1.0</kd>
-    <mu1>1000.0</mu1>
-    <mu2>1000.0</mu2>
-    <minDepth>0.001</minDepth>
   </gazebo>
 </robot>
